Commit message: -renamed packages

File: multi_rotors_description/urdf/multirotor_base.xacro (robot description, xacro)
@@ -81,5 +81,5 @@
         <geometry>
           <!-- <cylinder length="0.005" radius="${radius_rotor}"/> --> <!-- [m] -->
-          <!-- <mesh filename="package://rotors_description/meshes/propeller_${direction}.dae" -->
+          <!-- <mesh filename="package://multi_rotors_ftc_description/meshes/propeller_${direction}.dae" -->
           <mesh filename="package://multi_rotors_ftc_description/meshes/${mesh}_${direction}.dae"
             scale="${mesh_scale}" />
