Commit message: platform with failure and mass value changed

File: multi_rotors_description/urdf/ardrone_Normal.xacro (robot description, xacro)
@@ -7,5 +7,5 @@
   <xacro:property name="mesh_scale" value="0.001 0.001 0.001"/>
   <xacro:property name="mesh_scale_prop" value="0.001 0.001 0.001"/>
-  <xacro:property name="mass" value="0.6" /> <!-- [kg] -->
+  <xacro:property name="mass" value="1.5" /> <!-- [kg] -->
   <xacro:property name="body_width" value="0.3" /> <!-- [m] -->
   <xacro:property name="body_height" value="0.16" /> <!-- [m] -->
@@ -70,5 +70,5 @@
     mesh_scale="${mesh_scale_prop}"
     color="Red">
-    <origin xyz="-${sqrt2 * arm_length} -${sqrt2 * arm_length} ${rotor_offset_top}" rpy="0 0 0" />
+    <origin xyz="${sqrt2 * arm_length} -${sqrt2 * arm_length} ${rotor_offset_top}" rpy="0 0 0" />
     <xacro:insert_block name="rotor_inertia" />
   </xacro:vertical_rotor>
@@ -90,5 +90,5 @@
     mesh="ardrone_prop"
     mesh_scale="${mesh_scale_prop}"
-    color="blue">
+    color="DarkGrey">
     <origin xyz="-${sqrt2 * arm_length} ${sqrt2 * arm_length} ${rotor_offset_top}" rpy="0 0 0" />
     <xacro:insert_block name="rotor_inertia" />
@@ -131,5 +131,5 @@
     mesh_scale="${mesh_scale_prop}"
     color="DarkGrey">
-    <origin xyz="${sqrt2 * arm_length} -${sqrt2 * arm_length} ${rotor_offset_top}" rpy="0 0 0" />
+    <origin xyz="-${sqrt2 * arm_length} -${sqrt2 * arm_length} ${rotor_offset_top}" rpy="0 0 0" />
     <xacro:insert_block name="rotor_inertia" />
   </xacro:vertical_rotor>
