Commit message: - missing files

File: multi_rotors_description/urdf/ardrone.xacro (robot description, xacro)
@@ -38,5 +38,5 @@
   </xacro:property>
   <!-- Included URDF Files -->
-  <xacro:include filename="$(find rotors_description)/urdf/multirotor_base.xacro" />
+  <xacro:include filename="$(find multi_rotors_ftc_description)/urdf/multirotor_base.xacro" />
   <!-- Instantiate multirotor_base_macro once -->
   <xacro:multirotor_base_macro

File: multi_rotors_description/urdf/ardrone_base.xacro (robot description, xacro)
@@ -1,7 +1,7 @@
 <?xml version="1.0"?>
 <robot name="$(arg name)" xmlns:xacro="http://ros.org/wiki/xacro">
-  <xacro:include filename="$(find rotors_description)/urdf/component_snippets.xacro" />
+  <xacro:include filename="$(find multi_rotors_ftc_description)/urdf/component_snippets.xacro" />
   <!-- Instantiate ardrone "mechanics" -->
-  <xacro:include filename="$(find rotors_description)/urdf/ardrone.xacro" />
+  <xacro:include filename="$(find multi_rotors_ftc_description)/urdf/ardrone.xacro" />
   <!-- Instantiate a controller. -->
   <xacro:controller_plugin_macro

File: multi_rotors_description/urdf/component_snippets.xacro (robot description, xacro)
@@ -369,5 +369,5 @@
         <origin xyz="0 0 0" rpy="0 0 0" />
         <geometry>
-          <mesh filename="package://rotors_description/meshes/vi_sensor.dae" scale="1 1 1" />
+          <mesh filename="package://multi_rotors_ftc_description/meshes/vi_sensor.dae" scale="1 1 1" />
         </geometry>
       </visual>
@@ -550,5 +550,5 @@
         <origin xyz="-0.015 0.0035 0.004" rpy="${-pi/2} -${pi} ${-pi/2}"/>
         <geometry>
-          <mesh filename="package://rotors_description/meshes/asus_xtion_pro_live.dae" scale="0.001 0.001 0.001"/>
+          <mesh filename="package://multi_rotors_ftc_description/meshes/asus_xtion_pro_live.dae" scale="0.001 0.001 0.001"/>
         </geometry>
       </visual>
@@ -668,5 +668,5 @@
         <origin xyz="0 0 0" rpy="0 0 0" />
         <geometry>
-          <mesh filename="package://rotors_description/meshes/hokuyo.dae"/>
+          <mesh filename="package://multi_rotors_ftc_description/meshes/hokuyo.dae"/>
         </geometry>
       </visual>
@@ -674,5 +674,5 @@
 	<origin xyz="0 0 0" rpy="0 0 0" />
 	<geometry>
-	  <mesh filename="package://rotors_description/meshes/hokuyo.dae"/>
+	  <mesh filename="package://multi_rotors_ftc_description/meshes/hokuyo.dae"/>
 	</geometry>
       </collision>

File: multi_rotors_description/urdf/fati_ardrone_base.xacro (robot description, xacro)
@@ -355,5 +355,5 @@
         <origin xyz="0 0 0" rpy="0 0 0" />
         <geometry>
-          <mesh filename="package://rotors_description/meshes/vi_sensor.dae" scale="1 1 1" />
+          <mesh filename="package://multi_rotors_ftc_description/meshes/vi_sensor.dae" scale="1 1 1" />
         </geometry>
       </visual>
@@ -536,5 +536,5 @@
         <origin xyz="-0.015 0.0035 0.004" rpy="${-pi/2} -${pi} ${-pi/2}"/>
         <geometry>
-          <mesh filename="package://rotors_description/meshes/asus_xtion_pro_live.dae" scale="0.001 0.001 0.001"/>
+          <mesh filename="package://multi_rotors_ftc_description/meshes/asus_xtion_pro_live.dae" scale="0.001 0.001 0.001"/>
         </geometry>
       </visual>
@@ -654,5 +654,5 @@
         <origin xyz="0 0 0" rpy="0 0 0" />
         <geometry>
-          <mesh filename="package://rotors_description/meshes/hokuyo.dae"/>
+          <mesh filename="package://multi_rotors_ftc_description/meshes/hokuyo.dae"/>
         </geometry>
       </visual>
@@ -660,5 +660,5 @@
 	<origin xyz="0 0 0" rpy="0 0 0" />
 	<geometry>
-	  <mesh filename="package://rotors_description/meshes/hokuyo.dae"/>
+	  <mesh filename="package://multi_rotors_ftc_description/meshes/hokuyo.dae"/>
 	</geometry>
       </collision>
@@ -936,5 +936,5 @@
         <origin xyz="0 0 0" rpy="0 0 0" />
         <geometry>
-          <mesh filename="package://rotors_description/meshes/${mesh_file}"
+          <mesh filename="package://multi_rotors_ftc_description/meshes/${mesh_file}"
             scale="${mesh_scale}" />
           <!-- <box size="${body_width} ${body_width} ${body_height}"/> --> <!-- [m] [m] [m] -->
@@ -983,5 +983,5 @@
           <!-- <cylinder length="0.005" radius="${radius_rotor}"/> --> <!-- [m] -->
           <!-- <mesh filename="package://rotors_description/meshes/propeller_${direction}.dae" -->
-          <mesh filename="package://rotors_description/meshes/${mesh}_${direction}.dae"
+          <mesh filename="package://multi_rotors_ftc_description/meshes/${mesh}_${direction}.dae"
             scale="${mesh_scale}" />
           <!-- <box size="${2*radius_rotor} 0.01 0.005"/> -->

Commit message: multi_rotors_description/urdf/ardrone.xacro

File: multi_rotors_description/urdf/ardrone.xacro (robot description, xacro)
@@ -7,5 +7,5 @@
   <xacro:property name="mesh_scale" value="0.001 0.001 0.001"/>
   <xacro:property name="mesh_scale_prop" value="0.001 0.001 0.001"/>
-  <xacro:property name="mass" value="0.6" /> <!-- [kg] -->
+  <xacro:property name="mass" value="1.5" /> <!-- [kg] -->
   <xacro:property name="body_width" value="0.3" /> <!-- [m] -->
   <xacro:property name="body_height" value="0.16" /> <!-- [m] -->
@@ -18,5 +18,5 @@
   <xacro:property name="time_constant_up" value="0.0125" /> <!-- [s] -->
   <xacro:property name="time_constant_down" value="0.025" /> <!-- [s] -->
-  <xacro:property name="max_rot_velocity" value="838" /> <!-- [rad/s] -->
+  <xacro:property name="max_rot_velocity" value="1838" /> <!-- [rad/s] -->
   <xacro:property name="sin30" value="0.5" />
   <xacro:property name="cos30" value="0.866025403784" />
